File: eagle/mainboard/mainboard.sch (EAGLE design)
At the start: 45 parts, among them IC2 7805T, IC3 MEGA8-P, Q1 IRFZ48Z, Q2 IRFZ48Z, SW2 CT10-XXXX-G4, T1 BC547, T3 BC547

Commit message: RTC
Parts:
- added G1: CR2032V, battery:CR2032V
- added IC1: DS1302, ds1302:DS1302
- added Y1: 32,768kHz, special:XTAL/S
Connections:
- new net N$2: IC1.X1, Y1.2
- new net N$8: IC1.X2, Y1.1
- new net RTC_CLK: IC1.SCLK, IC3.PD2(INT0)
- new net RTC_IO: IC1.I/O, IC3.PD6(AIN0)
- new net RTC_RST: IC1.-RST, IC3.PD7(AIN1)
- new net VCC1: G1.+, IC1.VCC1
- net GND: now also G1.-, IC1.GND
- net VCC: now also IC1.VCC2
Other:
- moved on the sheet: JP1, JP13, JP4, JP5, JP6, JP7, JP8, JP9, R15, R16, R17, R2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
